File: hardware/TestBoard_ThermistorBreakout/ThermistorBreakoutPCB.kicad_sch (KiCad schematic)
At the start: 15 parts, among them J1 Conn_01x02, J2 Conn_01x03, J8 Conn_01x06

Commit message: redid thermistor board
Parts:
- removed J2: Conn_01x03, Connector_PinHeader_2.54mm:PinHeader_1x03_P2.54mm_Horizontal, symbol Connector_Generic:Conn_01x03
- removed R1, R2, R3, R4: 6.49k, Resistor_SMD:R_0603_1608Metric_Pad0.98x0.95mm_HandSolder, symbol Device:R
- removed TH1, TH2, TH3, TH4: Thermistor_NTC, UTSVT_Special:THERM_ERT-J1VR104FM, symbol Device:Thermistor_NTC
- removed TP1, TP2, TP3, TP4: TestPoint, TestPoint:TestPoint_Keystone_5005-5009_Compact, symbol Connector:TestPoint
- added TP10, TP11, TP8, TP9: TestPoint, TestPoint:TestPoint_Keystone_5005-5009_Compact, symbol Connector:TestPoint
Connections:
- net Temperature1: now also TP11.1
- net Temperature2: now also TP10.1
- net Temperature3: now also TP8.1
- net Temperature4: now also TP9.1
Other:
- added sheet Temperature1 (thermistorDivider.kicad_sch)
- added sheet Temperature2 (thermistorDivider.kicad_sch)
- added sheet Temperature3 (thermistorDivider.kicad_sch)
- added sheet Temperature4 (thermistorDivider.kicad_sch)
