File: hardware/VoltTemp/TemperatureFilter.kicad_sch (KiCad schematic)
At the start: 7 parts, among them U7 Opamp_Dual

Commit message: schematic mostly done
Parts:
- removed U7: Opamp_Dual, symbol Device:Opamp_Dual
- added C5: .1μF, Capacitor_SMD:C_0603_1608Metric_Pad1.08x0.95mm_HandSolder, symbol Device:C
- added TP11: TP_TempOut, TestPoint:TestPoint_Pad_1.0x1.0mm, symbol Connector:TestPoint
- added TP6: TP_TempIn, TestPoint:TestPoint_Pad_1.0x1.0mm, symbol Connector:TestPoint
- added U4: TLV9062xD, Package_SO:SOIC-8_3.9x4.9mm_P1.27mm, symbol Amplifier_Operational:TLV9062xD
- C25: footprint (none) -> Capacitor_SMD:C_0805_2012Metric_Pad1.18x1.45mm_HandSolder
- C3: renamed from C32; footprint (none) -> Capacitor_SMD:C_0805_2012Metric_Pad1.18x1.45mm_HandSolder
- R1: renamed from R49; footprint (none) -> Resistor_SMD:R_0603_1608Metric_Pad0.98x0.95mm_HandSolder
- R34, R35, R36: footprint (none) -> Resistor_SMD:R_0603_1608Metric_Pad0.98x0.95mm_HandSolder
Connections:
- net GNDA: now also C5.2, U4.4 (V-)
- net VDDA: now also C5.1, U4.8 (V+)
- net tempIn: now also TP6.1, U4.3 (+)
- net tempOut: now also TP11.1, U4.7
- net at C25.1, C3.1, R34.2: now also U4.5 (+)
- net at R35.2, R36.1: now also U4.6 (-)
- net at R1.1: now also U4.1, U4.2 (-)

Commit message: layout
Parts:
- removed TP6: TP_TempIn, TestPoint:TestPoint_Pad_1.0x1.0mm, symbol Connector:TestPoint
Changed lines of the file:
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@@
 	(paper "A4")
-	(junction
-		(at 59.69 58.42)
-		(diameter 0)
-		(color 0 0 0 0)
-	)
 	(junction
 		(at 82.55 83.82)
@@
 	(wire
 		(pts
-			(xy 57.15 58.42) (xy 59.69 58.42)
-		)
-		(stroke
-			(width 0)
-			(type default)
-		)
-	)
-	(wire
-		(pts
 			(xy 121.92 60.96) (xy 130.81 60.96)
 		)
@@
 	(wire
 		(pts
-			(xy 59.69 58.42) (xy 71.12 58.42)
-		)
-		(stroke
-			(width 0)
-			(type default)
-		)
-	)
-	(wire
-		(pts
-			(xy 59.69 57.15) (xy 59.69 58.42)
+			(xy 57.15 58.42) (xy 71.12 58.42)
 		)
 		(stroke
@@
 					(unit 1)
 				)
-			)
-		)
-	)
-	(symbol
-		(lib_id "Connector:TestPoint")
-		(at 59.69 57.15 0)
-		(unit 1)
-		(exclude_from_sim no)
-		(in_bom yes)
-		(on_board yes)
-		(dnp no)
-		(fields_autoplaced yes)
-		(property "Reference" "TP6"
-			(at 62.23 52.5779 0)
-			(effects
-				(font
-					(size 1.27 1.27)
-				)
-				(justify left)
-			)
-		)
-		(property "Value" "TP_TempIn"
-			(at 62.23 55.1179 0)
-			(effects
-				(font
-					(size 1.27 1.27)
-				)
-				(justify left)
-			)
-		)
-		(property "Footprint" "TestPoint:TestPoint_Pad_1.0x1.0mm"
-			(at 64.77 57.15 0)
-			(effects
-				(font
-					(size 1.27 1.27)
-				)
-				(hide yes)
-			)
-		)
-		(property "Datasheet" "~"
-			(at 64.77 57.15 0)
-			(effects
-				(font
-					(size 1.27 1.27)
-				)
-				(hide yes)
-			)
-		)
-		(property "Description" "test point"
-			(at 59.69 57.15 0)
-			(effects
-				(font
-					(size 1.27 1.27)
-				)
-				(hide yes)
-			)
-		)
-		(pin "1"
-		)
-		(instances
-			(project "BPS-Voltage_Temp_Board"
-				(path "/286f0d93-2a80-4abf-b115-d33410b730c4/b98a0b4d-b474-46e4-af8f-719e1bb91bc9/0071554d-4281-4843-9531-44fa66f109f1"
-					(reference "TP10")
-					(unit 1)
-				)
-				(path "/286f0d93-2a80-4abf-b115-d33410b730c4/b98a0b4d-b474-46e4-af8f-719e1bb91bc9/0b6a6f29-4cfd-471f-918e-165d9124c249"
-					(reference "TP8")
-					(unit 1)
-				)
-				(path "/286f0d93-2a80-4abf-b115-d33410b730c4/b98a0b4d-b474-46e4-af8f-719e1bb91bc9/305db25e-0e18-41b2-b157-490c9c9ed149"
-					(reference "TP6")
-					(unit 1)
-				)
-				(path "/286f0d93-2a80-4abf-b115-d33410b730c4/b98a0b4d-b474-46e4-af8f-719e1bb91bc9/4a5d6278-49ce-4bbe-b320-bfc4455852c3"
-					(reference "TP9")
-					(unit 1)
-				)
-				(path "/286f0d93-2a80-4abf-b115-d33410b730c4/b98a0b4d-b474-46e4-af8f-719e1bb91bc9/eab5a88a-8eae-40be-bde5-afb3b6331798"
-					(reference "TP7")
-					(unit 1)
-				)

Commit message: most layout done
Parts:
- C25: value C -> 1.2uF
- C3: value C -> 1uF; P/N (none) -> MLASU168SB5105KTNA01
- R1: value R -> 8.2kΩ
- R34: value R -> 27kΩ
- R35, R36: value R -> 2.7kΩ
Other:
- note added: "Assuming VDDA = 3.3V: At 10C, Rtherm = 226.2k ohms, tempOut = 184mV At 85C, Rtherm = 6.834k ohms, tempOut = 3.21V Very low temperature less than ~5C are seen as GND Very high temperatures greater than ~90C are seen as close to 3.3V Best solution will be achieved between 10C and 85C"
- note added: "tempIn is formed by a divider between a thermistor and 6.49k resistor"
- note added: "tempOut at 10C"
- note added: "tempOut at 85C"
- moved on the sheet: C25, C3, C5, R1, R34, R35, R36, TP11, U4A, U4B, U4C
