File: hardware/VoltTemp/TemperatureFilter.kicad_sch (KiCad schematic)
At the start: 9 parts, among them U4 TLV9062xD

Commit message: bom
Parts:
- C25: P/N (none) -> C0805C125K4RACTU
- C5: value .1μF -> 0.1uF
- R1: P/N (none) -> ERA-3AED822V
- R34: P/N (none) -> TNPU060327K0AYEN00
- R35, R36: P/N (none) -> SFR03EZPF2701
- U4: P/N (none) -> TLV9062QDGKRQ1
