File: hardware/VoltTemp/BPS-Voltage_Temp_Board.kicad_sch (KiCad schematic)
At the start: 22 parts, among them J10 53307-2471, J12 Conn_01x04, J13 Conn_01x04, J2 PeripheralCAN, J5 Logic_Analyzer

Commit message: bom
Parts:
- D14: P/N XL-1608UBC-06A -> NCD0603R1
