File: hardware/VoltTemp/VoltageConn.kicad_sch (KiCad schematic)
At the start: 27 parts, among them J11 Conn_01x07, J7 Conn_01x04

Commit message: bom
Parts:
- J11: P/N (none) -> 1053131107
- R23: P/N (none) -> SFR03EZPJ000
