File: hardware/VoltTemp/VoltageSense.kicad_sch (KiCad schematic)
At the start: 31 parts, among them IC1 ISO1641BDR, SW1 BOOT, U1 EL3H7, U2 BQ7692003PW, U3 EL3H7

Commit message: bom
Parts:
- C2: P/N TMK212BBJ106MGHT -> GRM21BR61H106KE43K
- C4: P/N 06033C471K4Z2A -> 06035C471J4Z2A
- R25, R26, R27, R28, R30: P/N (none) -> SFR03EZPJ000
- R5: P/N 667-ERJ-UP6D2001V -> CRCW06032K10FKEA
